File: Schematics/Overall/Master Device.brd (EAGLE design)
At the start: 50 x 90 mm, 38 parts, among them J1 POWER_JACK, U1 MPU-6050-1

Commit message: I'm not sure what changed. But here are changes.
Parts:
- added C12, C13: 22pF, SparkFun-Capacitors:0603
- added Y1: 16MHz, SparkFun-Clocks:HC49US
Connections:
- new net N$13: C13.2, MICROCONTROLLER.10, Y1.1
- new net N$15: C12.2, MICROCONTROLLER.9, Y1.2
- net GND: now also C12.1, C13.1
Routing:
- net N$13: track 0.00 -> 27.8 mm
- net N$15: track 0.00 -> 11.6 mm
- net GND: track 386.9 -> 395.2 mm
Changed lines of the file:
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@@
 <layers>
 <layer number="1" name="Top" color="4" fill="1" visible="yes" active="yes"/>
+<layer number="2" name="Route2" color="1" fill="3" visible="yes" active="yes"/>
+<layer number="3" name="Route3" color="4" fill="3" visible="yes" active="yes"/>
+<layer number="4" name="Route4" color="1" fill="4" visible="yes" active="yes"/>
+<layer number="5" name="Route5" color="4" fill="4" visible="yes" active="yes"/>
+<layer number="6" name="Route6" color="1" fill="8" visible="yes" active="yes"/>
+<layer number="7" name="Route7" color="4" fill="8" visible="yes" active="yes"/>
+<layer number="8" name="Route8" color="1" fill="2" visible="yes" active="yes"/>
+<layer number="9" name="Route9" color="4" fill="2" visible="yes" active="yes"/>
+<layer number="10" name="Route10" color="1" fill="7" visible="yes" active="yes"/>
+<layer number="11" name="Route11" color="4" fill="7" visible="yes" active="yes"/>
+<layer number="12" name="Route12" color="1" fill="5" visible="yes" active="yes"/>
+<layer number="13" name="Route13" color="4" fill="5" visible="yes" active="yes"/>
+<layer number="14" name="Route14" color="1" fill="6" visible="yes" active="yes"/>
+<layer number="15" name="Route15" color="4" fill="6" visible="yes" active="yes"/>
 <layer number="16" name="Bottom" color="1" fill="1" visible="yes" active="yes"/>
 <layer number="17" name="Pads" color="2" fill="1" visible="yes" active="yes"/>
@@
 <element name="U1" library="Testing" package="QFN-24-4MM2" value="MPU-6050-1" x="39.02" y="9.55" rot="R180"/>
 <element name="V_REG" library="SparkFun-IC-Power" package="78XXL" value="LD1117V33" x="18.86" y="10.65" rot="R180"/>
+<element name="Y1" library="SparkFun-Clocks" package="HC49US" value="16MHz" x="9" y="46" rot="R90">
+<attribute name="PROD_ID" value="XTAL-08181" x="9" y="46" size="1.778" layer="27" rot="R90" display="off"/>
+<attribute name="SF_ID" value="COM-00536" x="9" y="46" size="1.778" layer="27" rot="R90" display="off"/>
+</element>
+<element name="C12" library="SparkFun-Capacitors" package="0603" value="22pF" x="9.9" y="54.55" rot="R180">
+<attribute name="PROD_ID" value="CAP-07876" x="9.9" y="54.55" size="1.778" layer="27" rot="R180" display="off"/>
+</element>
+<element name="C13" library="SparkFun-Capacitors" package="0603" value="22pF" x="7.9" y="57.8" rot="R180">
+<attribute name="PROD_ID" value="CAP-07876" x="7.9" y="57.8" size="1.778" layer="27" rot="R180" display="off"/>
+</element>
 </elements>
 <signals>
@@
 <vertex x="1" y="-4.25"/>
 </polygon>
+<contactref element="C12" pad="1"/>
+<contactref element="C13" pad="1"/>
+<wire x1="8.75" y1="57.8" x2="10.75" y2="55.8" width="0.4064" layer="1"/>
+<wire x1="10.75" y1="55.8" x2="10.75" y2="54.55" width="0.4064" layer="1"/>
+<wire x1="10.75" y1="54.55" x2="13.55" y2="51.75" width="0.4064" layer="1"/>
+<wire x1="13.55" y1="51.75" x2="13.86" y2="51.75" width="0.4064" layer="1"/>
 </signal>
 <signal name="N$1">
@@
 <wire x1="37.66" y1="77.44" x2="42.01" y2="77.28" width="0.4064" layer="1"/>
 </signal>
+<signal name="N$13">
+<contactref element="Y1" pad="1"/>
+<contactref element="MICROCONTROLLER" pad="10"/>
+<contactref element="C13" pad="2"/>
+<wire x1="13.86" y1="46.67" x2="10.65" y2="43.46" width="0.4064" layer="1"/>
+<wire x1="10.65" y1="43.46" x2="9" y2="43.46" width="0.4064" layer="1"/>
+<wire x1="9" y1="43.46" x2="8.99" y2="43.45" width="0.4064" layer="1"/>
+<wire x1="8.99" y1="43.45" x2="4.5" y2="43.45" width="0.4064" layer="1"/>
+<wire x1="4.5" y1="43.45" x2="4.4" y2="43.55" width="0.4064" layer="1"/>
+<wire x1="4.4" y1="43.55" x2="4.4" y2="57.85" width="0.4064" layer="1"/>
+<wire x1="4.4" y1="57.85" x2="7.05" y2="57.8" width="0.4064" layer="1"/>
+</signal>
+<signal name="N$15">
+<contactref element="Y1" pad="2"/>
+<contactref element="MICROCONTROLLER" pad="9"/>
+<contactref element="C12" pad="2"/>
+<wire x1="13.86" y1="49.21" x2="9" y2="49.21" width="0.4064" layer="1"/>
+<wire x1="9" y1="49.21" x2="9" y2="48.54" width="0.4064" layer="1"/>
+<wire x1="9" y1="48.54" x2="9.05" y2="48.59" width="0.4064" layer="1"/>
+<wire x1="9.05" y1="48.59" x2="9.05" y2="54.55" width="0.4064" layer="1"/>
+</signal>
 </signals>
