File: Schematics/Overall/Master Device.brd (EAGLE design)
At the start: 50 x 90 mm, 38 parts, among them J1 POWER_JACK, U1 MPU-6050-1

Commit message: I'm not sure what changed. But here are changes.
Parts:
- added C12, C13: 22pF, SparkFun-Capacitors:0603
- added Y1: 16MHz, SparkFun-Clocks:HC49US
Connections:
- new net N$13: C13.2, MICROCONTROLLER.10, Y1.1
- new net N$15: C12.2, MICROCONTROLLER.9, Y1.2
- new net SD_CS: MICROCONTROLLER.16, SDCARD_READER.2
- net +3V3: no longer SDCARD_READER.2
- net GND: now also C12.1, C13.1
Routing:
- net N$13: track 0.00 -> 27.8 mm
- net SD_CS: track 0.00 -> 17.3 mm
- net N$15: track 0.00 -> 11.6 mm
- net GND: track 386.9 -> 395.2 mm
- net +3V3: track 249.8 -> 248.3 mm
Other:
- board size 50 x 90 mm -> 63 x 90 mm
Changed lines of the file:
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@@
 <layers>
 <layer number="1" name="Top" color="4" fill="1" visible="yes" active="yes"/>
+<layer number="2" name="Route2" color="1" fill="3" visible="yes" active="yes"/>
+<layer number="3" name="Route3" color="4" fill="3" visible="yes" active="yes"/>
+<layer number="4" name="Route4" color="1" fill="4" visible="yes" active="yes"/>
+<layer number="5" name="Route5" color="4" fill="4" visible="yes" active="yes"/>
+<layer number="6" name="Route6" color="1" fill="8" visible="yes" active="yes"/>
+<layer number="7" name="Route7" color="4" fill="8" visible="yes" active="yes"/>
+<layer number="8" name="Route8" color="1" fill="2" visible="yes" active="yes"/>
+<layer number="9" name="Route9" color="4" fill="2" visible="yes" active="yes"/>
+<layer number="10" name="Route10" color="1" fill="7" visible="yes" active="yes"/>
+<layer number="11" name="Route11" color="4" fill="7" visible="yes" active="yes"/>
+<layer number="12" name="Route12" color="1" fill="5" visible="yes" active="yes"/>
+<layer number="13" name="Route13" color="4" fill="5" visible="yes" active="yes"/>
+<layer number="14" name="Route14" color="1" fill="6" visible="yes" active="yes"/>
+<layer number="15" name="Route15" color="4" fill="6" visible="yes" active="yes"/>
 <layer number="16" name="Bottom" color="1" fill="1" visible="yes" active="yes"/>
 <layer number="17" name="Pads" color="2" fill="1" visible="yes" active="yes"/>
@@
 <board>
 <plain>
-<wire x1="0" y1="-5" x2="50" y2="-5" width="0" layer="20"/>
-<wire x1="50" y1="-5" x2="50" y2="85" width="0" layer="20"/>
-<wire x1="50" y1="85" x2="0" y2="85" width="0" layer="20"/>
-<wire x1="0" y1="85" x2="0" y2="-5" width="0" layer="20"/>
+<wire x1="-6" y1="-5" x2="57" y2="-5" width="0" layer="20"/>
+<wire x1="57" y1="-5" x2="57" y2="85" width="0" layer="20"/>
+<wire x1="57" y1="85" x2="-6" y2="85" width="0" layer="20"/>
+<wire x1="-6" y1="85" x2="-6" y2="-5" width="0" layer="20"/>
 <text x="48" y="36" size="1.778" layer="1" ratio="16" rot="R180">SD Reader</text>
 <text x="28" y="-2" size="1.016" layer="1" ratio="16">3.3V</text>
@@
 <element name="U1" library="Testing" package="QFN-24-4MM2" value="MPU-6050-1" x="39.02" y="9.55" rot="R180"/>
 <element name="V_REG" library="SparkFun-IC-Power" package="78XXL" value="LD1117V33" x="18.86" y="10.65" rot="R180"/>
+<element name="Y1" library="SparkFun-Clocks" package="HC49US" value="16MHz" x="9" y="46" rot="R90">
+<attribute name="PROD_ID" value="XTAL-08181" x="9" y="46" size="1.778" layer="27" rot="R90" display="off"/>
+<attribute name="SF_ID" value="COM-00536" x="9" y="46" size="1.778" layer="27" rot="R90" display="off"/>
+</element>
+<element name="C12" library="SparkFun-Capacitors" package="0603" value="22pF" x="9.9" y="54.55" rot="R180">
+<attribute name="PROD_ID" value="CAP-07876" x="9.9" y="54.55" size="1.778" layer="27" rot="R180" display="off"/>
+</element>
+<element name="C13" library="SparkFun-Capacitors" package="0603" value="22pF" x="7.9" y="57.8" rot="R180">
+<attribute name="PROD_ID" value="CAP-07876" x="7.9" y="57.8" size="1.778" layer="27" rot="R180" display="off"/>
+</element>
 </elements>
 <signals>
@@
 <wire x1="37.25" y1="14" x2="43" y2="14" width="0.3048" layer="16"/>
 <polygon width="0.3048" layer="16" isolate="1.27">
-<vertex x="1" y="84"/>
+<vertex x="-4" y="84"/>
 <vertex x="1.3" y="84.3"/>
 <vertex x="49.15" y="84.3"/>
-<vertex x="49.35" y="84.1"/>
-<vertex x="49.35" y="-4.35"/>
+<vertex x="55.35" y="84.1"/>
+<vertex x="55.35" y="-4.35"/>
 <vertex x="1.2" y="-4.35"/>
-<vertex x="1" y="-4.15"/>
+<vertex x="-4" y="-4.15"/>
 </polygon>
 <polygon width="0.4064" layer="1" isolate="1.27">
-<vertex x="1" y="84"/>
-<vertex x="49.35" y="84"/>
-<vertex x="49.35" y="81.5"/>
-<vertex x="49.4" y="81.5"/>
-<vertex x="49.4" y="-4.45"/>
+<vertex x="-4" y="84"/>
+<vertex x="55.35" y="84"/>
+<vertex x="55.35" y="81.5"/>
+<vertex x="55.4" y="81.5"/>
+<vertex x="55.4" y="-4.45"/>
 <vertex x="0.8" y="-4.45"/>
 <vertex x="0.8" y="-4.25"/>
-<vertex x="1" y="-4.25"/>
+<vertex x="-4" y="-4.25"/>
 </polygon>
+<contactref element="C12" pad="1"/>
+<contactref element="C13" pad="1"/>
+<wire x1="8.75" y1="57.8" x2="10.75" y2="55.8" width="0.4064" layer="1"/>
+<wire x1="10.75" y1="55.8" x2="10.75" y2="54.55" width="0.4064" layer="1"/>
+<wire x1="10.75" y1="54.55" x2="13.55" y2="51.75" width="0.4064" layer="1"/>
+<wire x1="13.55" y1="51.75" x2="13.86" y2="51.75" width="0.4064" layer="1"/>
 </signal>
 <signal name="N$1">
@@
 <contactref element="HC-05" pad="1"/>
 <contactref element="SDCARD_READER" pad="1"/>
-<contactref element="SDCARD_READER" pad="2"/>
 <contactref element="FSR2" pad="1"/>
 <contactref element="FSR1" pad="1"/>
@@
 <via x="21" y="30" extent="1-16" drill="0.6" shape="square"/>
 <wire x1="21" y1="30" x2="21" y2="30.94" width="0.6096" layer="16"/>
-<wire x1="21" y1="30.94" x2="25.8" y2="30.94" width="0.6096" layer="16"/>
-<wire x1="25.8" y1="30.94" x2="25.8" y2="33.48" width="0.6096" layer="16"/>
 <wire x1="25.8" y1="33.48" x2="34.43" y2="41" width="0.6096" layer="16"/>
 <wire x1="34.43" y1="41" x2="33.87" y2="52.12" width="0.6096" layer="1"/>
@@
 <wire x1="24" y1="46" x2="24" y2="49.21" width="0.6096" layer="16"/>
 <wire x1="24" y1="49.21" x2="21.48" y2="49.21" width="0.6096" layer="16"/>
+<wire x1="21" y1="30.94" x2="23.54" y2="33.48" width="0.6096" layer="16"/>
+<wire x1="23.54" y1="33.48" x2="25.8" y2="33.48" width="0.6096" layer="16"/>
 </signal>
 <signal name="TXA">
@@
 <wire x1="37.66" y1="77.44" x2="42.01" y2="77.28" width="0.4064" layer="1"/>
 </signal>
+<signal name="N$13">
+<contactref element="Y1" pad="1"/>
+<contactref element="MICROCONTROLLER" pad="10"/>
+<contactref element="C13" pad="2"/>
+<wire x1="13.86" y1="46.67" x2="10.65" y2="43.46" width="0.4064" layer="1"/>
+<wire x1="10.65" y1="43.46" x2="9" y2="43.46" width="0.4064" layer="1"/>
+<wire x1="9" y1="43.46" x2="8.99" y2="43.45" width="0.4064" layer="1"/>
+<wire x1="8.99" y1="43.45" x2="4.5" y2="43.45" width="0.4064" layer="1"/>
+<wire x1="4.5" y1="43.45" x2="4.4" y2="43.55" width="0.4064" layer="1"/>
+<wire x1="4.4" y1="43.55" x2="4.4" y2="57.85" width="0.4064" layer="1"/>
+<wire x1="4.4" y1="57.85" x2="7.05" y2="57.8" width="0.4064" layer="1"/>
+</signal>
+<signal name="N$15">
+<contactref element="Y1" pad="2"/>
+<contactref element="MICROCONTROLLER" pad="9"/>
+<contactref element="C12" pad="2"/>
+<wire x1="13.86" y1="49.21" x2="9" y2="49.21" width="0.4064" layer="1"/>
+<wire x1="9" y1="49.21" x2="9" y2="48.54" width="0.4064" layer="1"/>
+<wire x1="9" y1="48.54" x2="9.05" y2="48.59" width="0.4064" layer="1"/>
+<wire x1="9.05" y1="48.59" x2="9.05" y2="54.55" width="0.4064" layer="1"/>
+</signal>
+<signal name="SD_CS">
+<contactref element="SDCARD_READER" pad="2"/>
+<contactref element="MICROCONTROLLER" pad="16"/>
+<wire x1="21.48" y1="39.05" x2="20" y2="37.57" width="0.4064" layer="16"/>
+<wire x1="20" y1="37.57" x2="20" y2="29" width="0.4064" layer="16"/>
+<wire x1="20" y1="29" x2="23" y2="29" width="0.4064" layer="16"/>
+<wire x1="23" y1="29" x2="24.94" y2="30.94" width="0.4064" layer="16"/>
+<wire x1="24.94" y1="30.94" x2="25.8" y2="30.94" width="0.4064" layer="16"/>
+</signal>
 </signals>

Commit message: Hi
Other:
- board size 63 x 90 mm -> 62 x 90 mm
Changed lines of the file:
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@@
 <?xml version="1.0" encoding="utf-8"?>
 <!DOCTYPE eagle SYSTEM "eagle.dtd">
-<eagle version="8.1.0">
+<eagle version="8.0.1">
 <drawing>
 <settings>
@@
 <board>
 <plain>
-<wire x1="-6" y1="-5" x2="57" y2="-5" width="0" layer="20"/>
-<wire x1="57" y1="-5" x2="57" y2="85" width="0" layer="20"/>
-<wire x1="57" y1="85" x2="-6" y2="85" width="0" layer="20"/>
+<wire x1="-6" y1="-5" x2="56" y2="-5" width="0" layer="20"/>
+<wire x1="56" y1="-5" x2="56" y2="85" width="0" layer="20"/>
+<wire x1="56" y1="85" x2="-6" y2="85" width="0" layer="20"/>
 <wire x1="-6" y1="85" x2="-6" y2="-5" width="0" layer="20"/>
 <text x="48" y="36" size="1.778" layer="1" ratio="16" rot="R180">SD Reader</text>
@@
 <vertex x="1.3" y="84.3"/>
 <vertex x="49.15" y="84.3"/>
-<vertex x="55.35" y="84.1"/>
-<vertex x="55.35" y="-4.35"/>
+<vertex x="54.35" y="84.1"/>
+<vertex x="54.35" y="-4.35"/>
 <vertex x="1.2" y="-4.35"/>
 <vertex x="-4" y="-4.15"/>
@@
 <polygon width="0.4064" layer="1" isolate="1.27">
 <vertex x="-4" y="84"/>
-<vertex x="55.35" y="84"/>
-<vertex x="55.35" y="81.5"/>
-<vertex x="55.4" y="81.5"/>
-<vertex x="55.4" y="-4.45"/>
+<vertex x="54.35" y="84"/>
+<vertex x="54.35" y="81.5"/>
+<vertex x="54.4" y="81.5"/>
+<vertex x="54.4" y="-4.45"/>
 <vertex x="0.8" y="-4.45"/>
 <vertex x="0.8" y="-4.25"/>

Commit message: Gerber final round
Routing:
- net GND: track 395.2 -> 404.5 mm
Changed lines of the file:
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@@
 <wire x1="40.4" y1="67.27" x2="41.88" y2="65.79" width="0.6096" layer="1"/>
 <wire x1="41.88" y1="65.79" x2="41.88" y2="61.73" width="0.6096" layer="1"/>
-<wire x1="36.97" y1="43.96" x2="40.29" y2="47.28" width="0.6096" layer="16"/>
-<wire x1="36.97" y1="43.96" x2="36.97" y2="41" width="0.6096" layer="16"/>
+<wire x1="42.97" y1="43.96" x2="40.29" y2="47.28" width="0.6096" layer="16"/>
+<wire x1="42.97" y1="43.96" x2="36.97" y2="41" width="0.6096" layer="16"/>
 <wire x1="42.08" y1="16" x2="40.46" y2="15.38" width="0.6096" layer="1"/>
 <wire x1="43" y1="16" x2="46" y2="16" width="0.6096" layer="1"/>
@@
 <wire x1="13.86" y1="51.75" x2="16.4" y2="54.29" width="0.6096" layer="1"/>
 <wire x1="16.4" y1="54.29" x2="21.48" y2="54.29" width="0.6096" layer="1"/>
-<wire x1="36.97" y1="43.96" x2="36.93" y2="44" width="0.6096" layer="16"/>
+<wire x1="42.97" y1="43.96" x2="36.93" y2="44" width="0.6096" layer="16"/>
 <wire x1="29" y1="44" x2="29" y2="47" width="0.6096" layer="16"/>
 <wire x1="29" y1="47" x2="25" y2="47" width="0.6096" layer="16"/>
