File: Schematics/Overall/Master Device.sch (EAGLE design)
At the start: 30 parts, among them J1 POWER_JACK, U1 MPU-6050-1

Commit message: Updated Master with battery sensor
Parts:
- added NMOS: STN3NF06L, STN3NF06L:STN3NF06L
- added R14: 12K, resistor:R-US_R0805
- added R3: 500, resistor:R-US_R0805
- added R4: 20K, resistor:R-US_R0805
- added R5: 6K, resistor:R-US_R0805
Connections:
- removed net N$8: C1.1, J1.PWR, V_REG.IN
- new net 9V_BAT: C1.1, J1.PWR, R14.2, V_REG.IN
- new net N$12: NMOS.1, R3.2
- new net N$13: NMOS.2, R5.1
- new net SENSE: MICROCONTROLLER.PC2(ADC2), R14.1, R5.2
- new net V_MON: MICROCONTROLLER.PD4(XCK/T0), R3.1, R4.2
- net GND: now also NMOS.3, R4.1
Changed lines of the file:
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@@
 <?xml version="1.0" encoding="utf-8"?>
 <!DOCTYPE eagle SYSTEM "eagle.dtd">
-<eagle version="8.0.1">
+<eagle version="8.0.2">
 <drawing>
 <settings>
@@
 <part name="+3V16" library="supply1" deviceset="+3V3" device=""/>
 <part name="+3V18" library="supply1" deviceset="+3V3" device=""/>
+<part name="NMOS" library="STN3NF06L" deviceset="STN3NF06L" device=""/>
+<part name="GND5" library="supply1" deviceset="GND" device=""/>
+<part name="R3" library="resistor" deviceset="R-US_" device="R0805" value="500"/>
+<part name="R4" library="resistor" deviceset="R-US_" device="R0805" value="20K"/>
+<part name="GND6" library="supply1" deviceset="GND" device=""/>
+<part name="R5" library="resistor" deviceset="R-US_" device="R0805" value="6K"/>
+<part name="R14" library="resistor" deviceset="R-US_" device="R0805" value="12K"/>
 </parts>
 <sheets>
@@
 <instance part="+3V16" gate="G$1" x="180.34" y="149.86"/>
 <instance part="+3V18" gate="G$1" x="271.78" y="154.94"/>
+<instance part="NMOS" gate="A" x="263.84" y="68.58"/>
+<instance part="GND5" gate="1" x="270.46" y="52.96"/>
+<instance part="R3" gate="G$1" x="259.76" y="68.54"/>
+<instance part="R4" gate="G$1" x="254.76" y="60.54" rot="R90"/>
+<instance part="GND6" gate="1" x="254.54" y="51.42"/>
+<instance part="R5" gate="G$1" x="270" y="78.32" rot="R90"/>
+<instance part="R14" gate="G$1" x="270" y="91.02" rot="R90"/>
 </instances>
 <busses>
@@
 <wire x1="281.94" y1="127" x2="281.94" y2="111.76" width="0.1524" layer="91"/>
 </segment>
+<segment>
+<pinref part="NMOS" gate="A" pin="3"/>
+<pinref part="GND5" gate="1" pin="GND"/>
+<wire x1="270.825" y1="63.5" x2="270.46" y2="63.5" width="0.1524" layer="91"/>
+<wire x1="270.46" y1="63.5" x2="270.46" y2="55.5" width="0.1524" layer="91"/>
+</segment>
+<segment>
+<pinref part="GND6" gate="1" pin="GND"/>
+<pinref part="R4" gate="G$1" pin="1"/>
+<wire x1="254.54" y1="53.96" x2="254.76" y2="53.96" width="0.1524" layer="91"/>
+<wire x1="254.76" y1="53.96" x2="254.76" y2="55.46" width="0.1524" layer="91"/>
+</segment>
 </net>
 <net name="N$1" class="0">
@@
 </segment>
 </net>
-<net name="N$8" class="0">
+<net name="9V_BAT" class="0">
 <segment>
 <pinref part="C1" gate="G$1" pin="1"/>
@@
 <wire x1="129.54" y1="149.86" x2="137.16" y2="149.86" width="0.1524" layer="91"/>
 <junction x="129.54" y="149.86"/>
+<label x="129.54" y="149.86" size="1.016" layer="95" rot="R90" xref="yes"/>
+</segment>
+<segment>
+<pinref part="R14" gate="G$1" pin="2"/>
+<wire x1="270" y1="96.1" x2="269.24" y2="98.64" width="0.1524" layer="91"/>
+<label x="269.24" y="99.06" size="1.016" layer="95" xref="yes"/>
 </segment>
 </net>
@@
 </segment>
 </net>
+<net name="N$12" class="0">
+<segment>
+<pinref part="R3" gate="G$1" pin="2"/>
+<pinref part="NMOS" gate="A" pin="1"/>
+<wire x1="264.84" y1="68.54" x2="263.84" y2="68.54" width="0.1524" layer="91"/>
+<wire x1="263.84" y1="68.54" x2="263.84" y2="68.58" width="0.1524" layer="91"/>
+</segment>
+</net>
+<net name="SENSE" class="0">
+<segment>
+<pinref part="MICROCONTROLLER" gate="G$1" pin="PC2(ADC2)"/>
+<wire x1="165.1" y1="66.04" x2="170.18" y2="66.04" width="0.1524" layer="91"/>
+<label x="170.18" y="66.04" size="1.016" layer="95" xref="yes"/>
+</segment>
+<segment>
+<pinref part="R5" gate="G$1" pin="2"/>
+<pinref part="R14" gate="G$1" pin="1"/>
+<wire x1="270" y1="83.4" x2="270" y2="85.94" width="0.1524" layer="91"/>
+<label x="271.78" y="83.82" size="1.016" layer="95" xref="yes"/>
+</segment>
+</net>
+<net name="N$13" class="0">
+<segment>
+<pinref part="NMOS" gate="A" pin="2"/>
+<pinref part="R5" gate="G$1" pin="1"/>
+<wire x1="270.825" y1="73.66" x2="270" y2="73.66" width="0.1524" layer="91"/>
+<wire x1="270" y1="73.66" x2="270" y2="73.24" width="0.1524" layer="91"/>
+</segment>
+</net>
+<net name="V_MON" class="0">
+<segment>
+<pinref part="MICROCONTROLLER" gate="G$1" pin="PD4(XCK/T0)"/>
+<wire x1="165.1" y1="38.1" x2="170.18" y2="38.1" width="0.1524" layer="91"/>
+<label x="170.18" y="38.1" size="1.016" layer="95" xref="yes"/>
+</segment>
+<segment>
+<pinref part="R4" gate="G$1" pin="2"/>
+<pinref part="R3" gate="G$1" pin="1"/>
+<wire x1="254.76" y1="65.62" x2="254.68" y2="65.62" width="0.1524" layer="91"/>
+<wire x1="254.68" y1="65.62" x2="254.68" y2="68.54" width="0.1524" layer="91"/>
+<label x="254" y="68.58" size="1.016" layer="95" rot="R180" xref="yes"/>
+</segment>
+</net>

Commit message: Finalized Schematics
Parts:
- removed D2: RED, SparkFun-LED:LED3MM
- removed R14: 12K, resistor:R-US_R0805
- added C3: 10uF, SparkFun:CAP0603-CAP
- added C4: (no value), rcl:C-US050-050X075
- added D3: RED, SparkFun-LED:LED3MM
- added FSR1, FSR2: (no value), SparkFun-Connectors:CONN_02
- added MPU_BO: (no value), SparkFun-Connectors:CONN_05
- added R15: 68 Ohm, SparkFun-Resistors:68OHM-0603-1/10W-1%
- C1, C2: device SparkFun-Capacitors:0.1UF-KIT-EZ-50V-20% -> SparkFun:CAP0603-CAP
- C5: value 10uF -> (none); device SparkFun-Capacitors:10UF-1206-6.3V-20% -> rcl:C-US050-050X075
- PAIR/START, RESET: value MOMENTARY-SWITCH-SPST-PTH-6.0MM -> PTH-RIGHT; device SparkFun-Switches:MOMENTARY-SWITCH-SPST-PTH-6.0MM -> SparkFun-Switches:MOMENTARY-SWITCH-SPST-PTH-RIGHT-ANGLE-KIT
- R10, R11: value 20K -> 4k; device resistor:R-US_0411/15 -> SparkFun-Resistors:10KOHM-1/10W-1%(0603)0603
- R2: value 68 Ohm -> 4k; device SparkFun-Resistors:68OHM-0603-1/10W-1% -> SparkFun-Resistors:10KOHM-1/10W-1%(0603)0603
- R3: value 500 -> 20k; device resistor:R-US_R0805 -> SparkFun-Resistors:10KOHM-1/10W-1%(0603)0603
- R4: value 20K -> 500; device resistor:R-US_R0805 -> SparkFun-Resistors:10KOHM-1/10W-1%(0603)0603
- R5: value 6K -> 6k; device resistor:R-US_R0805 -> SparkFun-Resistors:10KOHM-1/10W-1%(0603)0603
- R8: value FSR -> 4k; device resistor:R-US_0204/5 -> SparkFun-Resistors:10KOHM-1/10W-1%(0603)0603
- R9: value FSR -> 12k; device resistor:R-US_0204/5 -> SparkFun-Resistors:10KOHM-1/10W-1%(0603)0603
Connections:
- removed net AUX_SCL: U1.AUX_CL
- removed net AUX_SDA: U1.AUX_DA
- removed net INT: U1.INT
- removed net N$12 (its old number): NMOS.1, R3.2
- new net MPU_INT: MICROCONTROLLER.PD2(INT0), MPU_BO.1, U1.INT
- new net N$11: NMOS.1, R4.1
- new net N$14: FSR2.2, R11.2, R8.2
- new net N$8: FSR1.2, R10.2, R2.2
- net +3V3: now also C2.1, C3.1, FSR1.1, FSR2.1, MPU_BO.5; no longer C5.1, R8.2, R9.2
- net 9V_BAT: now also R9.2; no longer R14.2
- net FSR1: now also C4.1, R10.1; no longer R10.2, R8.1
- net FSR2: now also C5.1, R11.1; no longer R11.2, R9.1
- net GND: now also C3.2, C4.2, D1.C, D3.C, MPU_BO.4, PAIR/START.1, R3.1, R8.1, RESET.1; no longer C2.1, PAIR/START.2, R1.1, R10.1, R11.1, R4.1, RESET.2
- net N$2: now also MICROCONTROLLER.PD3(INT1), RESET.2; no longer MICROCONTROLLER.PD2(INT0), RESET.1
- net N$3: now also PAIR/START.2; no longer PAIR/START.1
- net N$4: now also R1.2; no longer D2.A
- net N$5: now also R15.2; no longer D1.A
- net N$6: now also D3.A, R15.1; no longer D1.C, R1.2
- net N$7: now also D1.A, R1.1; no longer D2.C, R2.2
- net SCL: now also MPU_BO.2
- net SDA: now also MPU_BO.3
- net SENSE: now also R9.1; no longer R14.1
- net V_MON: now also R3.2; no longer R3.1
Other:
- moved on the sheet: C5, D1, NMOS, PAIR/START, R1, R10, R11, R2, R3, R4, R5, R6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

Commit message: worked on pcb layout
Parts:
- MPU_BO: value (none) -> MPU_BO
- SDCARD_READER: value (none) -> SD_READER
Changed lines of the file:
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@@
 <?xml version="1.0" encoding="utf-8"?>
 <!DOCTYPE eagle SYSTEM "eagle.dtd">
-<eagle version="8.0.2">
+<eagle version="7.6.0">
 <drawing>
 <settings>
@@
 <part name="+3V4" library="supply1" deviceset="+3V3" device=""/>
 <part name="+3V5" library="supply1" deviceset="+3V3" device=""/>
-<part name="SDCARD_READER" library="SparkFun-Connectors" deviceset="CONN_07" device=""/>
+<part name="SDCARD_READER" library="SparkFun-Connectors" deviceset="CONN_07" device="" value="SD_READER"/>
 <part name="+3V11" library="supply1" deviceset="+3V3" device=""/>
 <part name="GND13" library="supply1" deviceset="GND" device=""/>
@@
 <part name="RESET" library="SparkFun-Switches" deviceset="MOMENTARY-SWITCH-SPST" device="-PTH-RIGHT-ANGLE-KIT" value="PTH-RIGHT"/>
 <part name="PAIR/START" library="SparkFun-Switches" deviceset="MOMENTARY-SWITCH-SPST" device="-PTH-RIGHT-ANGLE-KIT" value="PTH-RIGHT"/>
-<part name="MPU_BO" library="SparkFun-Connectors" deviceset="CONN_05" device=""/>
+<part name="MPU_BO" library="SparkFun-Connectors" deviceset="CONN_05" device="" value="MPU_BO"/>
 </parts>
 <sheets>
@@
 <pinref part="MPU_BO" gate="G$1" pin="4"/>
 <wire x1="304.8" y1="127" x2="302.26" y2="127" width="0.1524" layer="91"/>
+<label x="302.26" y="127" size="1.016" layer="95" rot="R180" xref="yes"/>
 </segment>
 </net>
@@
 <pinref part="MPU_BO" gate="G$1" pin="3"/>
 <wire x1="304.8" y1="129.54" x2="302.26" y2="129.54" width="0.1524" layer="91"/>
+<label x="302.26" y="129.54" size="1.016" layer="95" rot="R180" xref="yes"/>
 </segment>
 </net>
@@
 <pinref part="MPU_BO" gate="G$1" pin="2"/>
 <wire x1="304.8" y1="132.08" x2="302.26" y2="132.08" width="0.1524" layer="91"/>
+<label x="302.26" y="132.08" size="1.016" layer="95" rot="R180" xref="yes"/>
 </segment>
 </net>
@@
 <pinref part="MPU_BO" gate="G$1" pin="5"/>
 <wire x1="304.8" y1="124.46" x2="302.26" y2="124.46" width="0.1524" layer="91"/>
+<label x="302.26" y="124.46" size="1.016" layer="95" rot="R180" xref="yes"/>
 </segment>
 </net>
@@
 <pinref part="MPU_BO" gate="G$1" pin="1"/>
 <wire x1="304.8" y1="134.62" x2="302.26" y2="134.62" width="0.1524" layer="91"/>
-</segment>
-</net>
+<label x="302.26" y="134.62" size="1.016" layer="95" rot="R180" xref="yes"/>
+</segment>
+</net>

Commit message: Added shape node to bottom for GND
Parts:
- removed SJ2, SJ3: SOLDERJUMPERTRACE, SparkFun:SOLDERJUMPERTRACE
Connections:
- removed net CLKIN: SJ2.2, U1.CLKIN
- removed net FSYNC: SJ3.2, U1.FSYNC
- net GND: now also U1.CLKIN, U1.FSYNC; no longer SJ2.1, SJ3.1
Changed lines of the file:
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@@
 <?xml version="1.0" encoding="utf-8"?>
 <!DOCTYPE eagle SYSTEM "eagle.dtd">
-<eagle version="7.6.0">
+<eagle version="8.1.0">
 <drawing>
 <settings>
@@
 <part name="GND23" library="SparkFun" deviceset="GND" device=""/>
 <part name="GND24" library="SparkFun" deviceset="GND" device=""/>
-<part name="SJ3" library="SparkFun" deviceset="SOLDERJUMPER" device="TRACE" value=""/>
-<part name="SJ2" library="SparkFun" deviceset="SOLDERJUMPER" device="TRACE" value=""/>
 <part name="+3V14" library="supply1" deviceset="+3V3" device=""/>
 <part name="+3V17" library="supply1" deviceset="+3V3" device=""/>
@@
 <instance part="GND23" gate="1" x="281.94" y="109.22"/>
 <instance part="GND24" gate="1" x="193.04" y="109.22"/>
-<instance part="SJ3" gate="1" x="193.04" y="119.38" rot="R90"/>
-<instance part="SJ2" gate="1" x="200.66" y="119.38" rot="R90"/>
 <instance part="+3V14" gate="G$1" x="289.56" y="154.94"/>
 <instance part="+3V17" gate="G$1" x="281.94" y="154.94"/>
@@
 <segment>
 <pinref part="GND22" gate="1" pin="GND"/>
-<wire x1="200.66" y1="111.76" x2="200.66" y2="114.3" width="0.1524" layer="91"/>
-<pinref part="SJ2" gate="1" pin="1"/>
+<pinref part="U1" gate="G$1" pin="CLKIN"/>
+<wire x1="226.06" y1="129.54" x2="200.66" y2="129.54" width="0.1524" layer="91"/>
+<label x="218.44" y="129.54" size="1.778" layer="95"/>
+<wire x1="200.66" y1="129.54" x2="200.66" y2="111.76" width="0.1524" layer="91"/>
 </segment>
 <segment>
 <pinref part="GND24" gate="1" pin="GND"/>
-<wire x1="193.04" y1="111.76" x2="193.04" y2="114.3" width="0.1524" layer="91"/>
-<pinref part="SJ3" gate="1" pin="1"/>
+<label x="218.44" y="132.08" size="1.778" layer="95"/>
+<pinref part="U1" gate="G$1" pin="FSYNC"/>
+<wire x1="193.04" y1="132.08" x2="226.06" y2="132.08" width="0.1524" layer="91"/>
+<wire x1="193.04" y1="132.08" x2="193.04" y2="111.76" width="0.1524" layer="91"/>
 </segment>
 <segment>
@@
 </segment>
 </net>
-<net name="FSYNC" class="0">
-<segment>
-<label x="218.44" y="132.08" size="1.778" layer="95"/>
-<pinref part="U1" gate="G$1" pin="FSYNC"/>
-<wire x1="193.04" y1="124.46" x2="193.04" y2="132.08" width="0.1524" layer="91"/>
-<wire x1="193.04" y1="132.08" x2="226.06" y2="132.08" width="0.1524" layer="91"/>
-<pinref part="SJ3" gate="1" pin="2"/>
-</segment>
-</net>
-<net name="CLKIN" class="0">
-<segment>
-<pinref part="U1" gate="G$1" pin="CLKIN"/>
-<wire x1="226.06" y1="129.54" x2="200.66" y2="129.54" width="0.1524" layer="91"/>
-<wire x1="200.66" y1="124.46" x2="200.66" y2="129.54" width="0.1524" layer="91"/>
-<label x="218.44" y="129.54" size="1.778" layer="95"/>
-<pinref part="SJ2" gate="1" pin="2"/>
-</segment>
-</net>

Commit message: I'm not sure what changed. But here are changes.
Parts:
- added C12, C13: 22pF, SparkFun-Capacitors:22PF-0603-50V-5%
- added Y1: 16MHz, SparkFun-Clocks:CRYSTAL-16MHZPTH-HC49US
Connections:
- new net N$13: C13.2, MICROCONTROLLER.PB7(XTAL2/TOSC2), Y1.1
- new net N$15: C12.2, MICROCONTROLLER.PB6(XTAL1/TOSC1), Y1.2
- new net SD_CS: MICROCONTROLLER.PB2(SS/OC1B), SDCARD_READER.2
- net +3V3: no longer SDCARD_READER.2
- net GND: now also C12.1, C13.1
Changed lines of the file:
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@@
 <part name="PAIR/START" library="SparkFun-Switches" deviceset="MOMENTARY-SWITCH-SPST" device="-PTH-RIGHT-ANGLE-KIT" value="PTH-RIGHT"/>
 <part name="MPU_BO" library="SparkFun-Connectors" deviceset="CONN_05" device="" value="MPU_BO"/>
+<part name="Y1" library="SparkFun-Clocks" deviceset="CRYSTAL-16MHZ" device="PTH-HC49US" value="16MHz"/>
+<part name="C12" library="SparkFun-Capacitors" deviceset="22PF" device="-0603-50V-5%" value="22pF"/>
+<part name="C13" library="SparkFun-Capacitors" deviceset="22PF" device="-0603-50V-5%" value="22pF"/>
 </parts>
 <sheets>
@@
 <instance part="PAIR/START" gate="G$1" x="210.82" y="25.4" rot="R90"/>
 <instance part="MPU_BO" gate="G$1" x="312.42" y="129.54" rot="R180"/>
+<instance part="Y1" gate="G$1" x="109.22" y="43.18" rot="R90"/>
+<instance part="C12" gate="G$1" x="106.68" y="45.72" rot="R90"/>
+<instance part="C13" gate="G$1" x="106.68" y="40.64" rot="R90"/>
 </instances>
 <busses>
@@
 <pinref part="MICROCONTROLLER" gate="G$1" pin="GND@1"/>
 <wire x1="116.84" y1="17.78" x2="106.68" y2="17.78" width="0.1524" layer="91"/>
+<wire x1="101.6" y1="45.72" x2="101.6" y2="40.64" width="0.1524" layer="91"/>
+<wire x1="101.6" y1="40.64" x2="101.6" y2="5.08" width="0.1524" layer="91"/>
+<wire x1="101.6" y1="5.08" x2="106.68" y2="5.08" width="0.1524" layer="91"/>
+<junction x="106.68" y="5.08"/>
+<pinref part="C12" gate="G$1" pin="1"/>
+<pinref part="C13" gate="G$1" pin="1"/>
+<junction x="101.6" y="40.64"/>
 </segment>
 <segment>
@@
 <wire x1="149.86" y1="119.38" x2="147.32" y2="119.38" width="0.1524" layer="91"/>
 <wire x1="147.32" y1="119.38" x2="147.32" y2="124.46" width="0.1524" layer="91"/>
-<pinref part="SDCARD_READER" gate="G$1" pin="2"/>
-<wire x1="149.86" y1="116.84" x2="147.32" y2="116.84" width="0.1524" layer="91"/>
-<wire x1="147.32" y1="116.84" x2="147.32" y2="119.38" width="0.1524" layer="91"/>
-<junction x="147.32" y="119.38"/>
 </segment>
 <segment>
@@
 </segment>
 </net>
+<net name="N$13" class="0">
+<segment>
+<pinref part="Y1" gate="G$1" pin="1"/>
+<pinref part="MICROCONTROLLER" gate="G$1" pin="PB7(XTAL2/TOSC2)"/>
+<wire x1="116.84" y1="40.64" x2="109.22" y2="40.64" width="0.1524" layer="91"/>
+<pinref part="C13" gate="G$1" pin="2"/>
+<junction x="109.22" y="40.64"/>
+</segment>
+</net>
+<net name="N$15" class="0">
+<segment>
+<pinref part="Y1" gate="G$1" pin="2"/>
+<pinref part="MICROCONTROLLER" gate="G$1" pin="PB6(XTAL1/TOSC1)"/>
+<wire x1="109.22" y1="45.72" x2="116.84" y2="45.72" width="0.1524" layer="91"/>
+<pinref part="C12" gate="G$1" pin="2"/>
+<junction x="109.22" y="45.72"/>
+</segment>
+</net>
+<net name="SD_CS" class="0">
+<segment>
+<pinref part="SDCARD_READER" gate="G$1" pin="2"/>
+<wire x1="149.86" y1="116.84" x2="142.24" y2="116.84" width="0.1524" layer="91"/>
+<label x="142.24" y="116.84" size="1.27" layer="95" rot="R180" xref="yes"/>
+</segment>
+<segment>
+<pinref part="MICROCONTROLLER" gate="G$1" pin="PB2(SS/OC1B)"/>
+<wire x1="165.1" y1="20.32" x2="170.18" y2="20.32" width="0.1524" layer="91"/>
+<label x="170.18" y="20.32" size="1.27" layer="95" xref="yes"/>
+</segment>
+</net>
