File: Schematics/Overall/Master Device.sch (EAGLE design)
At the start: 38 parts, among them J1 POWER_JACK, U1 MPU-6050-1

Commit message: I'm not sure what changed. But here are changes.
Parts:
- added C12, C13: 22pF, SparkFun-Capacitors:22PF-0603-50V-5%
- added Y1: 16MHz, SparkFun-Clocks:CRYSTAL-16MHZPTH-HC49US
Connections:
- new net N$13: C13.2, MICROCONTROLLER.PB7(XTAL2/TOSC2), Y1.1
- new net N$15: C12.2, MICROCONTROLLER.PB6(XTAL1/TOSC1), Y1.2
- net GND: now also C12.1, C13.1
Changed lines of the file:
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@@
 <part name="PAIR/START" library="SparkFun-Switches" deviceset="MOMENTARY-SWITCH-SPST" device="-PTH-RIGHT-ANGLE-KIT" value="PTH-RIGHT"/>
 <part name="MPU_BO" library="SparkFun-Connectors" deviceset="CONN_05" device="" value="MPU_BO"/>
+<part name="Y1" library="SparkFun-Clocks" deviceset="CRYSTAL-16MHZ" device="PTH-HC49US" value="16MHz"/>
+<part name="C12" library="SparkFun-Capacitors" deviceset="22PF" device="-0603-50V-5%" value="22pF"/>
+<part name="C13" library="SparkFun-Capacitors" deviceset="22PF" device="-0603-50V-5%" value="22pF"/>
 </parts>
 <sheets>
@@
 <instance part="PAIR/START" gate="G$1" x="210.82" y="25.4" rot="R90"/>
 <instance part="MPU_BO" gate="G$1" x="312.42" y="129.54" rot="R180"/>
+<instance part="Y1" gate="G$1" x="109.22" y="43.18" rot="R90"/>
+<instance part="C12" gate="G$1" x="106.68" y="45.72" rot="R90"/>
+<instance part="C13" gate="G$1" x="106.68" y="40.64" rot="R90"/>
 </instances>
 <busses>
@@
 <pinref part="MICROCONTROLLER" gate="G$1" pin="GND@1"/>
 <wire x1="116.84" y1="17.78" x2="106.68" y2="17.78" width="0.1524" layer="91"/>
+<wire x1="101.6" y1="45.72" x2="101.6" y2="40.64" width="0.1524" layer="91"/>
+<wire x1="101.6" y1="40.64" x2="101.6" y2="5.08" width="0.1524" layer="91"/>
+<wire x1="101.6" y1="5.08" x2="106.68" y2="5.08" width="0.1524" layer="91"/>
+<junction x="106.68" y="5.08"/>
+<pinref part="C12" gate="G$1" pin="1"/>
+<pinref part="C13" gate="G$1" pin="1"/>
+<junction x="101.6" y="40.64"/>
 </segment>
 <segment>
@@
 </segment>
 </net>
+<net name="N$13" class="0">
+<segment>
+<pinref part="Y1" gate="G$1" pin="1"/>
+<pinref part="MICROCONTROLLER" gate="G$1" pin="PB7(XTAL2/TOSC2)"/>
+<wire x1="116.84" y1="40.64" x2="109.22" y2="40.64" width="0.1524" layer="91"/>
+<pinref part="C13" gate="G$1" pin="2"/>
+<junction x="109.22" y="40.64"/>
+</segment>
+</net>
+<net name="N$15" class="0">
+<segment>
+<pinref part="Y1" gate="G$1" pin="2"/>
+<pinref part="MICROCONTROLLER" gate="G$1" pin="PB6(XTAL1/TOSC1)"/>
+<wire x1="109.22" y1="45.72" x2="116.84" y2="45.72" width="0.1524" layer="91"/>
+<pinref part="C12" gate="G$1" pin="2"/>
+<junction x="109.22" y="45.72"/>
+</segment>
+</net>
